File: robot_za_sledenje_crti.kicad_pcb (KiCad board)
At the start: 2 copper layers, 102.9 x 102.9 mm, 34 parts, among them M1 Motor_Encoder, M2 Motor_Encoder, Q1 Q_NPN_BCE, SW1 SWITCH

Commit message: Add files via upload
Parts:
- moved MICROCONTROLLER1 48.5 mm to (143.5, 128.3), turned to 90 degrees
- moved MC1 30.5 mm to (153.7, 104.1), turned to 270 degrees
Connections:
- net ENCDB renamed Net-(M1-Pad5)
- net ENCLB renamed Net-(M2-Pad5)
- net XOR-D renamed Net-(MICROCONTROLLER1-Pad24)
- net XOR-L renamed Net-(MICROCONTROLLER1-Pad25)
- BT1 pad 1: (no net) -> Net-(BT1-Pad1)
- BT1 pad 2: (no net) -> Net-(BT1-Pad2)
- BT1 pad 3: (no net) -> GND
- BT1 pad 4: (no net) -> +5V
- MICROCONTROLLER1 pad 10: (no net) -> PWML1
- MICROCONTROLLER1 pad 11: (no net) -> PWML2
- MICROCONTROLLER1 pad 12: (no net) -> S0
- MICROCONTROLLER1 pad 13: (no net) -> S1
- MICROCONTROLLER1 pad 2: (no net) -> Net-(MICROCONTROLLER1-Pad2)
- MICROCONTROLLER1 pad 3: (no net) -> Net-(BT1-Pad1)
- MICROCONTROLLER1 pad 4: (no net) -> Net-(BT1-Pad2)
- MICROCONTROLLER1 pad 5: (no net) -> Net-(MICROCONTROLLER1-Pad5)
- MICROCONTROLLER1 pad 6: (no net) -> Net-(MICROCONTROLLER1-Pad6)
- MICROCONTROLLER1 pad 7: (no net) -> ENCLA
- MICROCONTROLLER1 pad 8: (no net) -> ENCDA
- MICROCONTROLLER1 pad 9: (no net) -> QR-ON
