File: robot_za_sledenje_crti.sch (KiCad schematic (older format))
At the start: 29 parts

Commit message: Add files via upload
Parts:
- removed BT?: BT-RN42, symbol BT-RN42
- added BT?: JY-MCU, symbol JY-MCU
- added BT?: Battery_Cell, symbol Battery_Cell
- added R1k: R, symbol R
- added SW?: SWITCH, symbol SWITCH
Connections:
- net +5V: now also BT?.4 (VCC)
- net +9V: now also BT?.1 (+)
- net ENCDA: now also M?.~ (VCC), MICROCONTROLLER?.7 (2/SDA), XOR?.1 (A)
- net ENCDB: now also M?.~ (VCC), MICROCONTROLLER?.22 (A1), XOR?.2 (B)
- net GND: now also BT?.3 (GND), SW?.2
- net QR-ON: now also R1k.2; no longer Q?.1 (B)
- net at MICROCONTROLLER?.3 (1/TX): now also BT?.1 (RX-I)
- net at MICROCONTROLLER?.4 (0/RX): now also BT?.2 (TX-0)
- removed net ENCLA: M?.~ (VCC), MICROCONTROLLER?.7 (2/SDA), XOR?.1 (A)
- removed net ENCLB: M?.~ (VCC), MICROCONTROLLER?.22 (A1), XOR?.2 (B)
- new net: Q?.1 (B), R1k.1
- new net: BT?.2 (-), SW?.1
Other:
- moved on the sheet: XOR?
Changed lines of the file:
@@
 F 1 "Q_NPN_BCE" H 1400 6550 50  0000 L CNN
 F 2 "" H 1400 6700 50  0000 C CNN
-F 3 "" H 1200 6600 50  0000 C CNN
+F 3 "http://www.farnell.com/datasheets/2195017.pdf?_ga=1.266460878.1717627041.1488214545" H 1200 6600 50  0001 C CNN
 	1    1200 6600
 	1    0    0    -1
@@
 Text Label 9100 2150 0    60   ~ 0
 PWML1
-Text GLabel 3800 2250 0    60   Input ~ 0
+Text GLabel 3300 2250 0    60   Input ~ 0
 PWML1
-Text GLabel 4200 2350 0    60   Input ~ 0
+Text GLabel 3700 2350 0    60   Input ~ 0
 PWML2
-Text GLabel 3800 2650 0    60   Input ~ 0
+Text GLabel 3300 2650 0    60   Input ~ 0
 PWMD1
-Text GLabel 4200 2750 0    60   Input ~ 0
+Text GLabel 3700 2750 0    60   Input ~ 0
 PWMD2
 Text GLabel 8200 2600 3    60   Input ~ 0
@@
 Wire Wire Line
 	8100 2150 8100 1000
-Text GLabel 4200 1950 0    60   Input ~ 0
+Text GLabel 3650 1950 0    60   Input ~ 0
 ENCLA
-Text GLabel 3800 2050 0    60   Input ~ 0
+Text GLabel 3300 2050 0    60   Input ~ 0
 ENCDA
 Text GLabel 9700 2600 3    60   Input ~ 0
@@
 Text GLabel 7850 2600 3    60   Input ~ 0
 ENCDA
-Text GLabel 1000 6600 0    60   Input ~ 0
+Text GLabel 950  7100 0    60   Input ~ 0
 QR-ON
-Text GLabel 4200 2150 0    60   Input ~ 0
+Text GLabel 3700 2150 0    60   Input ~ 0
 QR-ON
 Wire Wire Line
@@
 Wire Wire Line
 	2350 4150 2600 4150
-Text GLabel 3800 2450 0    60   Input ~ 0
+Text GLabel 3100 2450 0    60   Input ~ 0
 S0
-Text GLabel 4200 2550 0    60   Input ~ 0
+Text GLabel 3500 2550 0    60   Input ~ 0
 S1
-Text GLabel 4200 2950 0    60   Input ~ 0
+Text GLabel 3500 2950 0    60   Input ~ 0
 S2
 Wire Wire Line
-	3800 2050 4200 2050
-Wire Wire Line
-	4200 2250 3800 2250
-Wire Wire Line
-	3800 2450 4200 2450
-Wire Wire Line
-	4200 2650 3800 2650
+	3300 2050 4200 2050
+Wire Wire Line
+	3300 2250 4200 2250
+Wire Wire Line
+	3100 2450 4200 2450
+Wire Wire Line
+	3300 2650 4200 2650
 $Comp
 L +9V #PWR?
@@
 Wire Wire Line
 	3600 1200 3600 1650
-$Comp
-L BT-RN42 BT?
-U 1 1 58C51963
-P 3750 1500
-F 0 "BT?" H 3150 1300 51  0000 C CNN
-F 1 "BT-RN42" H 3150 2200 51  0000 C CNN
-F 2 "" H 3600 1350 10  0001 C CNN
-F 3 "" H 3550 1400 10  0001 C CNN
-	1    3750 1500
-	1    0    0    -1
-$EndComp
 Wire Wire Line
 	3800 1550 3800 1400
@@
 Wire Wire Line
 	9850 1600 9850 1100
-Text GLabel 5650 2550 2    60   Input ~ 0
+Text GLabel 6650 2550 2    60   Input ~ 0
 ENCLB
-Text GLabel 6000 2450 2    60   Input ~ 0
+Text GLabel 6650 2450 2    60   Input ~ 0
 ENCDB
 Wire Wire Line
-	5650 2450 6000 2450
+	5650 2450 6650 2450
 $Comp
 L XOR-Gate XOR?
 U 1 1 58C56B38
-P 7750 4300
-F 0 "XOR?" H 7800 4100 60  0000 C CNN
-F 1 "XOR-Gate" H 7800 4500 60  0000 C CNN
-F 2 "" H 7800 4100 60  0001 C CNN
-F 3 "http://uk.farnell.com/texas-instruments/sn74lvc1g86dbvr/ic-ex-or-single-2-input-smd/dp/1287521" H 7800 4100 60  0001 C CNN
-	1    7750 4300
+P 5100 4150
+F 0 "XOR?" H 5150 3950 60  0000 C CNN
+F 1 "XOR-Gate" H 5150 4350 60  0000 C CNN
+F 2 "" H 5150 3950 60  0001 C CNN
+F 3 "http://uk.farnell.com/texas-instruments/sn74lvc1g86dbvr/ic-ex-or-single-2-input-smd/dp/1287521" H 5150 3950 60  0001 C CNN
+	1    5100 4150
 	1    0    0    -1
 $EndComp
@@
 L XOR-Gate XOR?
 U 1 1 58C56C27
-P 9550 4300
-F 0 "XOR?" H 9600 4100 60  0000 C CNN
-F 1 "XOR-Gate" H 9600 4500 60  0000 C CNN
-F 2 "" H 9600 4100 60  0001 C CNN
-F 3 "http://uk.farnell.com/texas-instruments/sn74lvc1g86dbvr/ic-ex-or-single-2-input-smd/dp/1287521" H 9600 4100 60  0001 C CNN
-	1    9550 4300
+P 5100 4850
+F 0 "XOR?" H 5150 4650 60  0000 C CNN
+F 1 "XOR-Gate" H 5150 5050 60  0000 C CNN
+F 2 "" H 5150 4650 60  0001 C CNN
+F 3 "http://uk.farnell.com/texas-instruments/sn74lvc1g86dbvr/ic-ex-or-single-2-input-smd/dp/1287521" H 5150 4650 60  0001 C CNN
+	1    5100 4850
 	1    0    0    -1
 $EndComp
@@
 L +5V #PWR?
 U 1 1 58C56FE0
-P 9950 4200
-F 0 "#PWR?" H 9950 4050 50  0001 C CNN
-F 1 "+5V" H 9950 4340 50  0000 C CNN
-F 2 "" H 9950 4200 50  0000 C CNN
-F 3 "" H 9950 4200 50  0000 C CNN
-	1    9950 4200
+P 5500 4750
+F 0 "#PWR?" H 5500 4600 50  0001 C CNN
+F 1 "+5V" H 5500 4890 50  0000 C CNN
+F 2 "" H 5500 4750 50  0000 C CNN
+F 3 "" H 5500 4750 50  0000 C CNN
+	1    5500 4750
 	1    0    0    -1
 $EndComp
@@
 L +5V #PWR?
 U 1 1 58C57272
+P 5500 4050
+F 0 "#PWR?" H 5500 3900 50  0001 C CNN
+F 1 "+5V" H 5500 4190 50  0000 C CNN
+F 2 "" H 5500 4050 50  0000 C CNN
+F 3 "" H 5500 4050 50  0000 C CNN
+	1    5500 4050
+	1    0    0    -1
+$EndComp
+$Comp
+L GND #PWR?
+U 1 1 58C59941
+P 4800 4250
+F 0 "#PWR?" H 4800 4000 50  0001 C CNN
+F 1 "GND" H 4800 4100 50  0000 C CNN
+F 2 "" H 4800 4250 50  0000 C CNN
+F 3 "" H 4800 4250 50  0000 C CNN
+	1    4800 4250
+	1    0    0    -1
+$EndComp
+$Comp
+L GND #PWR?
+U 1 1 58C59C5B
+P 4800 4950
+F 0 "#PWR?" H 4800 4700 50  0001 C CNN
+F 1 "GND" H 4800 4800 50  0000 C CNN
+F 2 "" H 4800 4950 50  0000 C CNN
+F 3 "" H 4800 4950 50  0000 C CNN
+	1    4800 4950
+	1    0    0    -1
+$EndComp
+Text GLabel 5500 4250 2    60   Input ~ 0
+XOR-D
+Text GLabel 6650 2350 2    60   Input ~ 0
+XOR-D
+Text GLabel 5500 4950 2    60   Input ~ 0
+XOR-L
+Text GLabel 6650 2250 2    60   Input ~ 0
+XOR-L
+Wire Wire Line
+	5650 2250 6650 2250
+Wire Wire Line
+	4200 1950 3650 1950
+Wire Wire Line
+	4200 2150 3700 2150
+Wire Wire Line
+	3700 2350 4200 2350
+Wire Wire Line
+	4200 2550 3500 2550
+Wire Wire Line
+	4200 2750 3700 2750
+Wire Wire Line
+	3500 2950 4200 2950
+Wire Wire Line
+	4200 2050 4200 4050
+Wire Wire Line
+	4200 4050 4800 4050
+Wire Wire Line
+	6650 2350 5650 2350
+Wire Wire Line
+	5650 2550 6650 2550
+Wire Wire Line
+	4800 4150 4800 3700
+Wire Wire Line
+	4800 3700 5650 3700
+Wire Wire Line
+	5650 3700 5650 2450
+Wire Wire Line
+	4800 4750 4200 4750
+Wire Wire Line
+	4200 4750 4200 1950
+Wire Wire Line
+	4800 4850 4800 4500
+Wire Wire Line
+	4800 4500 5650 4500
+Wire Wire Line
+	5650 4500 5650 2550
+$Comp
+L R R1k
+U 1 1 58CF9223
+P 1000 6750
+F 0 "R1k" V 1080 6750 50  0000 C CNN
+F 1 "R" V 1000 6750 50  0000 C CNN
+F 2 "" V 930 6750 50  0000 C CNN
+F 3 "" H 1000 6750 50  0000 C CNN
+	1    1000 6750
+	1    0    0    -1
+$EndComp
+Wire Wire Line
+	1000 6900 1000 7100
+Wire Wire Line
+	1000 7100 950  7100
+$Comp
+L JY-MCU BT?
+U 1 1 58CFD3F7
+P 3150 1250
+F 0 "BT?" H 3150 1000 51  0000 C CNN
+F 1 "JY-MCU" H 3200 1500 51  0000 C CNN
+F 2 "" H 3600 850 10  0001 C CNN
+F 3 "" H 3550 900 10  0001 C CNN
+	1    3150 1250
+	1    0    0    -1
+$EndComp
+$Comp
+L Battery_Cell BT?
+U 1 1 58CFE501
+P 7800 4100
+F 0 "BT?" H 7900 4200 50  0000 L CNN
+F 1 "Battery_Cell" H 7900 4100 50  0000 L CNN
+F 2 "" V 7800 4160 50  0000 C CNN
+F 3 "" V 7800 4160 50  0000 C CNN
+	1    7800 4100
+	1    0    0    -1
+$EndComp
+$Comp
+L +9V #PWR?
+U 1 1 58CFE574
+P 7800 3900
+F 0 "#PWR?" H 7800 3750 50  0001 C CNN
+F 1 "+9V" H 7800 4040 50  0000 C CNN
+F 2 "" H 7800 3900 50  0000 C CNN
+F 3 "" H 7800 3900 50  0000 C CNN
+	1    7800 3900
+	1    0    0    -1
+$EndComp
+$Comp
+L SWITCH SW?
+U 1 1 58CFE72F
 P 8150 4200
-F 0 "#PWR?" H 8150 4050 50  0001 C CNN
-F 1 "+5V" H 8150 4340 50  0000 C CNN
-F 2 "" H 8150 4200 50  0000 C CNN
-F 3 "" H 8150 4200 50  0000 C CNN
+F 0 "SW?" H 8150 4100 60  0000 C CNN
+F 1 "SWITCH" H 8200 4400 60  0000 C CNN
+F 2 "" H 8150 4200 60  0001 C CNN
+F 3 "http://si.farnell.com/erg-components/jsa4-1-g0/switch-jumper-1-way-spst-slide/dp/3289758" H 8150 4200 60  0001 C CNN
 	1    8150 4200
 	1    0    0    -1
 $EndComp
-Text GLabel 7450 4200 0    60   Input ~ 0
-ENCDA
-Text GLabel 7450 4300 0    60   Input ~ 0
-ENCDB
-$Comp
-L GND #PWR?
-U 1 1 58C59941
-P 7450 4400
-F 0 "#PWR?" H 7450 4150 50  0001 C CNN
-F 1 "GND" H 7450 4250 50  0000 C CNN
-F 2 "" H 7450 4400 50  0000 C CNN
-F 3 "" H 7450 4400 50  0000 C CNN
-	1    7450 4400
-	1    0    0    -1
-$EndComp
-$Comp
-L GND #PWR?
-U 1 1 58C59C5B
-P 9250 4400
-F 0 "#PWR?" H 9250 4150 50  0001 C CNN
-F 1 "GND" H 9250 4250 50  0000 C CNN
-F 2 "" H 9250 4400 50  0000 C CNN
-F 3 "" H 9250 4400 50  0000 C CNN
-	1    9250 4400
-	1    0    0    -1
-$EndComp
-Text GLabel 9250 4200 0    60   Input ~ 0
-ENCLA
-Text GLabel 9250 4300 0    60   Input ~ 0
-ENCLB
-Text GLabel 8150 4400 2    60   Input ~ 0
-XOR-D
-Text GLabel 5650 2350 2    60   Input ~ 0
-XOR-D
-Text GLabel 9950 4400 2    60   Input ~ 0
-XOR-L
-Text GLabel 6000 2250 2    60   Input ~ 0
-XOR-L
-Wire Wire Line
-	5650 2250 6000 2250
+$Comp
+L GND #PWR?
+U 1 1 58CFE7D8
+P 8550 4200
+F 0 "#PWR?" H 8550 3950 50  0001 C CNN
+F 1 "GND" H 8550 4050 50  0000 C CNN
+F 2 "" H 8550 4200 50  0000 C CNN
+F 3 "" H 8550 4200 50  0000 C CNN
+	1    8550 4200
+	1    0    0    -1
+$EndComp
 $EndSCHEMATC

Commit message: Add files via upload
Parts:
- removed 10k (x7): R, symbol R
- removed M?: MOTOR-L, symbol MOTOR-L
- removed M?: MOTOR-D, symbol MOTOR-D
- removed R?: 150, symbol R
- added 2R150: R, komponentefp:R150, symbol R
- added M1, M2: Motor_Encoder, komponentefp:EM_Encoder, symbol Motor_Encoder
- added R10k2, R10k3, R10k4, R10k5, R10k6, R10k7, R10k8: R, komponentefp:R10k, symbol R
- 1R150: renamed from R?; value 150 -> R; footprint (none) -> komponentefp:R150
- BT1: renamed from BT?; footprint (none) -> komponentefp:JY_MCU
- BT2: renamed from BT?; footprint (none) -> komponentefp:Baterry
- C1, C2: footprint (none) -> Capacitors_ThroughHole:C_Radial_D5_L6_P2.5
- MC1: renamed from MC?; footprint (none) -> komponentefp:L293_MOTOR_CONTROLLER
- MICROCONTROLLER1: renamed from MICROCONTROLLER?; footprint (none) -> komponentefp:ARDUINO_MICRO_SHIELD
- MUX1: renamed from MUX; footprint (none) -> komponentefp:mux4051
- Q1: renamed from Q?; footprint (none) -> komponentefp:npn-10v
- QR1, QR2, QR3, QR4, QR5, QR6, QR7, QR8: footprint (none) -> komponentefp:QRE1113
- R10k1: renamed from 10k; footprint (none) -> komponentefp:R10k
- R1k1: renamed from R1k; footprint (none) -> komponentefp:R1k
- SW1: renamed from SW?; footprint (none) -> komponentefp:switch
- XOR1, XOR2: renamed from XOR?; footprint (none) -> komponentefp:XOR-GATE
Connections:
- net +5V: now also M1.3 (VCC), M2.3 (VCC), R10k2.1, R10k3.1, R10k4.1, R10k5.1, R10k6.1, R10k7.1, R10k8.1
- net +9V: now also 2R150.1
- net ENCDA: now also M1.4 (OUT-A); no longer MICROCONTROLLER1.7 (2/SDA), XOR2.1 (A)
- net ENCDB: now also M1.5 (OUT-B); no longer MICROCONTROLLER1.22 (A1), XOR2.2 (B)
- net GND: now also M1.6 (GND), M2.6 (GND)
- net at MUX1.14 (X1), QR2.3 (C): now also R10k2.2
- net at MUX1.15 (X2), QR3.3 (C): now also R10k3.2
- net at MUX1.12 (X3), QR4.3 (C): now also R10k4.2
- net at QR5.1 (A+): now also 2R150.2
- net at MUX1.1 (X4), QR5.3 (C): now also R10k5.2
- net at MUX1.5 (X5), QR6.3 (C): now also R10k6.2
- net at MUX1.2 (X6), QR7.3 (C): now also R10k7.2
- net at MUX1.4 (X7), QR8.3 (C): now also R10k8.2
- net at C2.1, MC1.11 (3Y): now also M2.1 (M1)
- net at C2.2, MC1.14 (4Y): now also M2.2 (M2)
- net at C1.1, MC1.3 (1Y): now also M1.1 (M1)
- net at C1.2, MC1.6 (2Y): now also M1.2 (M2)
- new net ENCLA: M2.4 (OUT-A), MICROCONTROLLER1.7 (2/SDA), XOR2.1 (A)
- new net ENCLB: M2.5 (OUT-B), MICROCONTROLLER1.22 (A1), XOR2.2 (B)
- no-connect marks 0 -> 12
